File: Digital out expander/Digital out expander.kicad_sch (KiCad schematic)
At the start: 126 parts, among them J1 Screw_Terminal_01x03, J10 Conn_01x03_Pin, J11 Conn_01x03_Pin, J12 Conn_01x03_Pin, J13 Conn_01x03_Pin, J14 Conn_01x03_Pin, J15 Conn_01x03_Pin, J16 Conn_01x03_Pin, J17 Conn_01x03_Pin, J18 Screw_Terminal_01x16, J19 Conn_01x04_Pin, J2 Conn_01x03_Pin, J20 Conn_01x04_Pin, J21 Conn_01x04_Pin, J22 Conn_01x04_Pin, J23 Conn_01x04_Pin, J24 Conn_01x03_Pin, J3 Conn_01x03_Pin, J4 Conn_01x03_Pin, J5 Conn_01x03_Pin, J6 Conn_01x03_Pin, J7 Conn_01x03_Pin, J8 Conn_01x03_Pin, J9 Conn_01x03_Pin, Q1 2N5401, Q10 2N5401, Q11 2N5401, Q12 2N5401, Q13 2N5401, Q14 2N5401, Q15 2N5401, Q16 2N5401, Q17 BC547, Q18 BC547, Q19 BC547, Q2 2N5401, Q20 BC547, Q21 BC547, Q22 BC547, Q23 BC547, Q24 BC547, Q25 BC547, Q26 BC547, Q27 BC547, Q28 BC547, Q29 BC547, Q3 2N5401, Q30 BC547, Q31 BC547, Q32 BC547, Q4 2N5401, Q5 2N5401, Q6 2N5401, Q7 2N5401, Q8 2N5401, Q9 2N5401, U1 PC847, U2 PC847, U3 PC847, U4 PC847, U5 MCP23017_SO

Commit message: Nu borde det fungera bättre
Connections:
- net at R48.2: now also C1.1, J19.1 (Pin_1), J19.2 (Pin_2), J19.3 (Pin_3), J19.4 (Pin_4), J22.1 (Pin_1), J23.1 (Pin_1), R33.2, R34.2, R35.2, R36.2, R37.2, R38.2, R39.2, R40.2, R41.2, R42.2, R43.2, R44.2, R45.2, R46.2, R47.2, U5.9 (VDD); no longer Q32.3 (E)
- net at Q21.3 (E): now also C1.2, J21.1 (Pin_1), J21.2 (Pin_2), J21.3 (Pin_3), J21.4 (Pin_4), J22.2 (Pin_2), J23.2 (Pin_2), Q17.3 (E), Q18.3 (E), Q19.3 (E), Q20.3 (E), Q22.3 (E), Q23.3 (E), Q24.3 (E), Q25.3 (E), Q26.3 (E), Q27.3 (E), Q28.3 (E), Q29.3 (E), Q30.3 (E), Q31.3 (E), Q32.3 (E), U5.10 (VSS); no longer R37.2
- new net: Q28.1 (C), U3.8
- new net: Q24.1 (C), U2.8
- new net: Q26.1 (C), U3.4
- new net: Q31.1 (C), U4.6
- new net: Q30.1 (C), U4.4
- new net: Q17.1 (C), U1.2
- new net: Q27.1 (C), U3.6
- new net: Q23.1 (C), U2.6
- new net: Q18.1 (C), U1.4
- new net: Q22.1 (C), U2.4
- new net: Q19.1 (C), U1.6
- new net: Q21.1 (C), U2.2
- new net: Q29.1 (C), U4.2
- new net: Q20.1 (C), U1.8
- new net: Q32.1 (C), U4.8
- new net: Q25.1 (C), U3.2
Other:
- moved on the sheet: Q17, Q18, Q19, Q20, Q21, Q22, Q23, Q24, Q25, Q26, Q27, Q28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

Commit message: Förbättrad läsbarhet
Other:
- moved on the sheet: C1, J19, J20, J21, J22, J23, J24, R49, R50, R51, R52, R53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

Commit message: Fixat ordning på bitarna
Connections:
- net at J7.2 (Pin_2), R6.1: now also Q6.1 (E); no longer Q6.2 (E)
- net at R22.1, R6.2: now also Q6.2 (B); no longer Q6.1 (B)
- net at R55.2: now also U5.27 (GPA6); no longer U5.7 (GPB6)
- net at R61.2: now also U5.5 (GPB4); no longer U5.25 (GPA4)
- net at J5.2 (Pin_2), R4.1: now also Q4.1 (E); no longer Q4.2 (E)
- net at J14.2 (Pin_2), R13.1: now also Q13.1 (E); no longer Q13.2 (E)
- net at R13.2, R29.1: now also Q13.2 (B); no longer Q13.1 (B)
- net at R19.1, R3.2: now also Q3.2 (B); no longer Q3.1 (B)
- net at J4.2 (Pin_2), R3.1: now also Q3.1 (E); no longer Q3.2 (E)
- net at R58.2: now also U5.2 (GPB1); no longer U5.22 (GPA1)
- net at J11.2 (Pin_2), R10.1: now also Q10.1 (E); no longer Q10.2 (E)
- net at R10.2, R26.1: now also Q10.2 (B); no longer Q10.1 (B)
- net at R11.2, R27.1: now also Q11.2 (B); no longer Q11.1 (B)
- net at J12.2 (Pin_2), R11.1: now also Q11.1 (E); no longer Q11.2 (E)
- net at R20.1, R4.2: now also Q4.2 (B); no longer Q4.1 (B)
- net at J17.2 (Pin_2), R16.1: now also Q16.1 (E); no longer Q16.2 (E)
- net at R16.2, R32.1: now also Q16.2 (B); no longer Q16.1 (B)
- net at J13.2 (Pin_2), R12.1: now also Q12.1 (E); no longer Q12.2 (E)
- net at R12.2, R28.1: now also Q12.2 (B); no longer Q12.1 (B)
- net at R25.1, R9.2: now also Q9.2 (B); no longer Q9.1 (B)
- net at J10.2 (Pin_2), R9.1: now also Q9.1 (E); no longer Q9.2 (E)
- net at R57.2: now also U5.1 (GPB0); no longer U5.21 (GPA0)
- net at R60.2: now also U5.4 (GPB3); no longer U5.24 (GPA3)
- net at R64.2: now also U5.8 (GPB7); no longer U5.28 (GPA7)
- net at J3.2 (Pin_2), R2.1: now also Q2.1 (E); no longer Q2.2 (E)
- net at R18.1, R2.2: now also Q2.2 (B); no longer Q2.1 (B)
- net at R59.2: now also U5.3 (GPB2); no longer U5.23 (GPA2)
- net at R24.1, R8.2: now also Q8.2 (B); no longer Q8.1 (B)
- net at J9.2 (Pin_2), R8.1: now also Q8.1 (E); no longer Q8.2 (E)
- net at R50.2: now also U5.22 (GPA1); no longer U5.2 (GPB1)
- net at R49.2: now also U5.21 (GPA0); no longer U5.1 (GPB0)
- net at U5.26 (GPA5): now also R54.2; no longer R62.2
- net at R63.2: now also U5.7 (GPB6); no longer U5.27 (GPA6)
- net at R51.2: now also U5.23 (GPA2); no longer U5.3 (GPB2)
- net at R52.2: now also U5.24 (GPA3); no longer U5.4 (GPB3)
- net at R53.2: now also U5.25 (GPA4); no longer U5.5 (GPB4)
- net at U5.6 (GPB5): now also R62.2; no longer R54.2
- net at R56.2: now also U5.28 (GPA7); no longer U5.8 (GPB7)
- net at J2.2 (Pin_2), R1.1: now also Q1.1 (E); no longer Q1.2 (E)
- net at R1.2, R17.1: now also Q1.2 (B); no longer Q1.1 (B)
- net at R21.1, R5.2: now also Q5.2 (B); no longer Q5.1 (B)
- net at J16.2 (Pin_2), R15.1: now also Q15.1 (E); no longer Q15.2 (E)
- net at J8.2 (Pin_2), R7.1: now also Q7.1 (E); no longer Q7.2 (E)
- net at R23.1, R7.2: now also Q7.2 (B); no longer Q7.1 (B)
- net at R14.2, R30.1: now also Q14.2 (B); no longer Q14.1 (B)
- net at J15.2 (Pin_2), R14.1: now also Q14.1 (E); no longer Q14.2 (E)
- net at R15.2, R31.1: now also Q15.2 (B); no longer Q15.1 (B)
- net at J6.2 (Pin_2), R5.1: now also Q5.1 (E); no longer Q5.2 (E)
Other:
- moved on the sheet: C1, J19, J20, J21, J22, J23, J24, U5

Commit message: Ändrade jumpers för bättre tydlighet
Parts:
- removed J19, J20, J21: Conn_01x04_Pin, symbol Connector:Conn_01x04_Pin
- added J19, J20, J21, J22: Conn_01x03_Pin, symbol Connector:Conn_01x03_Pin
- renumbered J22 to J23, J23 to J24, J24 to J25
Connections:
- net at C1.1, J23.1 (Pin_1), J24.1 (Pin_1)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: now also J19.1 (Pin_1), J20.1 (Pin_1), J21.1 (Pin_1), J22.1 (Pin_1)
- net at C1.2, J23.2 (Pin_2), J24.2 (Pin_2)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: now also J19.3 (Pin_3), J20.3 (Pin_3), J21.3 (Pin_3), J22.3 (Pin_3)
- net at U5.15 (A0): now also J19.2 (Pin_2)
- net at U5.16 (A1): now also J20.2 (Pin_2)
- net at U5.17 (A2): now also J21.2 (Pin_2)
- net at J25.3 (Pin_3), U5.18 (~{RESET}): now also J22.2 (Pin_2)
Other:
- moved on the sheet: C1
